File: V5/esp-24v-16ch-v5-i2c.kicad_sch (KiCad schematic)
At the start: 24 parts, among them J9 SENSORS, SW2 1WIRE_SEL, U6 MCP23008-xSS, U7 MCP23008-xSS, U8 MCP23017_SS, U9 DS2482S-100

Commit message: V6 is up
Parts:
- removed C28, C29, C32, C34, C37: 10uF/25V, Tales:C_0805_2012Metric, symbol Device:C_Small
- removed C31: 100nF/50V, Tales:C_0402_1005Metric, symbol Device:C_Small
- removed R37: 1k, Tales:R_0402_1005Metric, symbol Device:R_US
- removed U6, U7: MCP23008-xSS, Package_SO:SSOP-20_5.3x7.2mm_P0.65mm, symbol Interface_Expansion:MCP23008-xSS
- added C63: 10uF/10V, Tales:C_0603_1608Metric, symbol Device:C_Small
- added R136, R137: 10k, Tales:R_0402_1005Metric, symbol Device:R_US
- added U6: MCP23017_SS, Package_SO:SSOP-28_5.3x10.2mm_P0.65mm, symbol Interface_Expansion:MCP23017_SS
- C29: renamed from C35; Package (none) -> 0402/1005
- C64: renamed from C30; Package (none) -> 0402/1005
- renumbered C36 to C28, C33 to C62, D8 to D73, D9 to D8, J9 to J4, R40 to R37, U8 to U7, U9 to U8
Connections:
- net +3V3: now also U6.9 (VDD)
- net +5V: now also C63.1
- net GND: now also C63.2, R136.2, R137.2, U6.10 (VSS), U6.15 (A0), U6.16 (A1), U6.17 (A2)
- net I2CSCL: now also U6.12 (SCK)
- net I2CSDA: now also U6.13 (SDA)
- net IN10: now also U6.1 (GPB0)
- net IN11: now also U6.2 (GPB1)
- net IN12: now also U6.3 (GPB2)
- net IN13: now also U6.4 (GPB3)
- net IN14: now also U6.5 (GPB4)
- net IN15: now also U6.6 (GPB5)
- net IN16: now also U6.7 (GPB6)
- net IN3: now also U6.21 (GPA0)
- net IN4: now also U6.22 (GPA1)
- net IN5: now also U6.23 (GPA2)
- net IN6: now also U6.24 (GPA3)
- net IN7: now also U6.25 (GPA4)
- net IN8: now also U6.26 (GPA5)
- net IN9: now also U6.27 (GPA6)
- net MCPINN1RST renamed MCPINNRST
- net MCPINNRST: now also U6.18 (~{RESET})
- new net GPA7: R136.1, U6.28 (GPA7)
- new net GPB7: R137.1, U6.8 (GPB7)
- new net MCPININTA: U6.20 (INTA)
- new net MCPININTB: U6.19 (INTB)
Other:
- note added: "PINS GPA7 E GPB7 ON THE MCP23017 MUST NOT BE USED AS INPUTS TIE THEM TO GND VIA PULLDOWN RESISTOR AND CONFIGURE AS UNUSED IN THE TEMPLATE"
- note removed: "INPUTS ADDRESS 0x21"
- moved on the sheet: C27, C28, R36, R37, U7
