File: V6/esp-24v-16ch-v6-power.kicad_sch (KiCad schematic)
At the start: 38 parts, among them J1 VIN, J2 USB_C_Receptacle_USB2.0, Q1 WPM2015-3/TR, Q2 MMUN2211LT3G, U1 TX4138, U2 SY8089A1AAC

Commit message: V6 is up
Parts:
- removed C12: 10uF/10V, Tales:C_0603_1608Metric, symbol Device:C_Small
- added C11: 10uF/25V, Tales:C_0805_2012Metric, symbol Device:C_Small
- C1: renamed from C8; value 10uF/10V -> 10uF/25V; footprint Tales:C_0603_1608Metric -> Tales:C_0805_2012Metric; Case 0603/1608 -> 0805/2012; LCSC Part # C19702 -> C15850; Mfr PN CL10A106KP8NNNC -> CL21A106KAYNNNE; Package 0603/1608 -> (none); Vendor PN C19702 -> C15850
- C10: renamed from C4; Technology Ceramic -> Ceramic C0G
- C12: renamed from C5; Package D8xL10.5mm -> (none)
- C3: renamed from C2; Package 0402/1005 -> (none)
- C4: renamed from C9; Package 0402/1005 -> (none)
- C5: renamed from C6; Package 0402/1005 -> (none)
- C6: renamed from C7; Package 0402/1005 -> (none)
- C7: renamed from C10; Package 1206/3216 -> (none)
- C8: renamed from C11; Package 1206/3216 -> (none)
- C9: renamed from C3; Package 0805/2012 -> (none)
- J6: renamed from J1; footprint Tales:TerminalBlock_Dibo_DB142V-5.08-2P_1x02_P5.08mm_Vertical -> Tales:TerminalBlock_Wago_250-202_1x02_P3.5mm_45Degree; LCSC Part # C2898699 -> C2765061; Mfr Dorabo -> Wago; Mfr PN DB142V-5.08-2P -> 250-202; Vendor PN C2898699 -> C2765061
- R10: renamed from R3; Package 0603/1608 -> (none)
- R11: renamed from R4; Package 0603/1608 -> (none)
- R2: renamed from R5; Package 0402/1005 -> (none)
- R3: renamed from R6; Package 0402/1005 -> (none)
- R6: renamed from R1; Package 1206/3216 -> (none)
- R7: renamed from R2; Package 0603/1608 -> (none)
- R8: renamed from R10; Package 0402/1005 -> (none)
- renumbered C1 to C2, D6 to D1, D1 to D2, D4 to D3, D5 to D4, D2 to D5, D3 to D6, J2 to J7, L2 to L1, L1 to L2, R7 to R1, R8 to R4, R9 to R5, R11 to R9, U2 to U1, U1 to U2
Connections:
- net +3V3LAN: now also C11.1
- net GND: now also C11.2
