File: V6/esp-24v-16ch-v6.kicad_pcb (KiCad board)
At the start: 4 copper layers, 128 x 67.8 mm, 327 parts, among them J1 ENTRADAS 1-8, J2 GNDIO, J3 ENTRADAS 9-16, J4 SAÍDAS 1-8, J5 SAÍDAS 9-16, J6 VIN, J7 USB_C_Receptacle_USB2.0, J8 ETHERNET, J9 SENSORS, Q1 WPM2015-3/TR, Q10 MMBT2222A, Q11 MMBT2222A, Q12 MMBT2222A, Q13 MMBT2222A, Q14 MMBT2222A, Q15 MMBT2222A, Q16 MMBT2222A, Q17 MMBT2222A, Q18 MMBT2222A, Q19 MMBT2222A, Q2 MMUN2211LT3G, Q3 UMH3N, Q4 MMBT2222A, Q5 MMBT2222A, Q6 MMBT2222A, Q7 MMBT2222A, Q8 MMBT2222A, Q9 MMBT2222A, SW1 RESET, SW2 1WIRE_SEL, U1 SY8089A1AAC, U10 OR-3H7-4, U11 OR-3H7-4, U12 OR-3H7-4, U13 OR-3H7-4, U2 TX4138, U3 CH340K, U4 ESP32-WROOM-32UE-N16, U5 LAN8710A, U6 MCP23008-xSS, U7 MCP23008-xSS, U8 MCP23017x-x-SS, U9 DS2482S-100

Commit message: Revising power rails
Parts:
- removed the C21 at (182.8, 99.3)
- added C12: 100nF/50V, Tales:C_0402_1005Metric, F.Cu at (164.8, 95.6)
- added C14: 10uF/25V, Tales:C_0805_2012Metric, F.Cu at (169.3, 97.3)
- added TP1: GND, TestPoint:TestPoint_Pad_D1.5mm, F.Cu at (143.3, 131.8)
- added TP2: 5V, TestPoint:TestPoint_Pad_D1.5mm, F.Cu at (155.8, 97.4)
- added TP3: 3V3, TestPoint:TestPoint_Pad_D1.5mm, F.Cu at (144.3, 98.8)
- added TP4: 3V3LAN, TestPoint:TestPoint_Pad_D1.5mm, F.Cu at (182.5, 60.1)
- added TP5: 3V3A, TestPoint:TestPoint_Pad_D1.5mm, F.Cu at (167.8, 109.6)
- moved R22 24.0 mm to (167.0, 126.6), turned to 90 degrees
- moved R24 8.93 mm to (174.0, 106.1), turned to 90 degrees
- moved C25 1.12 mm to (171.8, 96.8), turned to 90 degrees
- moved L3 0.75 mm to (166.3, 96.1)
- moved C11 0.25 mm to (163.3, 96.1)
- renumbered C12 to C13, C13 to C15, C14 to C16, C15 to C17, C16 to C18, C17 to C19, C18 to C20, C19 to C21, C20 to C22, C22 to C23, C23 to C24, C24 to C25, C25 to C26, C26 to C27, C27 to C28, C29 to C30, C30 to C31, C31 to C32, C33 to C34, C34 to C35, C35 to C36, C36 to C37, C37 to C38, C38 to C39, C39 to C40, C40 to C41, C41 to C42, C42 to C43, C43 to C44, C44 to C45, C45 to C46, C46 to C47, C47 to C48, C48 to C49, C49 to C50, C50 to C51, C51 to C52, C52 to C53, C53 to C54, C54 to C55, C55 to C56, C56 to C57, C57 to C58, C58 to C59, C59 to C60, C60 to C61, C61 to C62, C62 to C63, C63 to C64, C64 to C65, C65 to C66, C66 to C67, C67 to C68, C68 to C69, C69 to C70, R25 to R20, R20 to R24, R24 to R25
Connections:
- J8 pad 10: /LAN/ETHLEDGK -> /LAN/ETHLEDYK
- J8 pad 11: /LAN/ETHLEDYA -> /LAN/ETHLEDGA
- J8 pad 12: GND -> /LAN/ETHLEDGK
- J8 pad 9: /LAN/ETHLEDGA -> +3V3A
- R22 pad 1: /LAN/ETHLEDY -> /LAN/ETHLEDGK
- R22 pad 2: /LAN/ETHLEDYA -> GND
- R24 pad 1: +3V3LAN -> /LAN/ETHLEDYK
- R24 pad 2: /LAN/ETHLEDGA -> /LAN/ETHLEDY
- U5 pad 2: /LAN/ETHLEDGK -> /LAN/ETHLEDY
- U5 pad 3: /LAN/ETHLEDY -> /LAN/ETHLEDGA
Routing:
- net /LAN/ETHLEDYA: track 34.7 -> 0.00 mm, vias 1 -> 0
- net /LAN/ETHLEDGK: track 31.7 -> 2.55 mm
- net /LAN/ETHLEDYK: track 0.00 -> 26.5 mm
- net /LAN/ETHLEDGA: track 19.8 -> 37.2 mm, vias 0 -> 1
- net +3V3A: track 14.6 -> 30.0 mm, vias 6 -> 8
- net GND: track 136.6 -> 144.3 mm, vias 132 -> 133
- net /LAN/ETHLEDY: track 1.80 -> 4.16 mm
- net +3V3LAN: track 22.0 -> 20.8 mm, vias 7 -> 6

Commit message: Update esp-24v-16ch-v6.kicad_pcb
Parts:
- moved TP4 45.0 mm to (183.3, 105.1)
Routing:
- net +3V3LAN: track 20.8 -> 22.8 mm
- net /LAN/EMACCLK: track 48.0 -> 49.0 mm
Changed lines of the file:
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@@
 			(unit
 				(name "A")
-				(pins "3" "4" "5" "21" "22" "17" "18" "20" "19" "32" "2" "1" "38" "39"
-					"15" "25" "35" "24" "34" "26" "29" "14" "16" "13" "23" "27" "28" "30"
+				(pins "3" "4" "5" "21" "22" "17" "18" "20" "19" "32" "2" "1" "38" "15"
+					"39" "25" "35" "24" "34" "26" "29" "14" "16" "13" "23" "27" "28" "30"
 					"31" "33" "36" "37" "10" "11" "12" "8" "9" "6" "7"
 				)
@@
 		(tags "resistor")
 		(property "Reference" "R28"
-			(at -2 0 0)
+			(at 0 -1.25 0)
 			(layer "F.SilkS")
 			(effects
@@
 	(footprint "TestPoint:TestPoint_Pad_D1.5mm"
 		(layer "F.Cu")
-		(at 182.545 60.105)
+		(at 183.27 105.08)
 		(descr "SMD pad as test Point, diameter 1.5mm")
 		(tags "test point SMD pad")
 		(property "Reference" "TP4"
-			(at 0 -1.648 0)
+			(at 0.25 1.75 0)
 			(layer "F.SilkS")
 			(effects
 				(font
-					(size 1 1)
-					(thickness 0.15)
+					(size 0.8 0.6)
+					(thickness 0.1)
+					(bold yes)
 				)
 			)
@@
 		(tags "test point SMD pad")
 		(property "Reference" "TP5"
-			(at -1.25 1.25 0)
+			(at -1.5 1.5 0)
 			(layer "F.SilkS")
 			(effects
@@
 		(tags "resistor")
 		(property "Reference" "R29"
-			(at -2 0 0)
+			(at 1 1 0)
 			(layer "F.SilkS")
 			(effects
@@
 	)
 	(segment
-		(start 167.27 97.1425)
-		(end 166.27 97.1425)
-		(width 0.5)
-		(layer "F.Cu")
-		(net "+3V3A")
-	)
-	(segment
 		(start 173.77 102.08)
 		(end 173.77 102.35)
@@
 	)
 	(segment
+		(start 167.27 97.1425)
+		(end 166.27 97.1425)
+		(width 0.5)
+		(layer "F.Cu")
+		(net "+3V3A")
+	)
+	(segment
 		(start 171.77 98.08)
 		(end 172.02 98.33)
@@
 	)
 	(segment
+		(start 182.53 104.34)
+		(end 182.53 103.33)
+		(width 0.5)
+		(layer "F.Cu")
+		(net "+3V3LAN")
+	)
+	(segment
 		(start 164.77 95.1)
 		(end 164.25 95.1)
@@
 	)
 	(segment
+		(start 183.27 105.08)
+		(end 182.53 104.34)
+		(width 0.5)
+		(layer "F.Cu")
+		(net "+3V3LAN")
+	)
+	(segment
 		(start 165.25 95.1)
 		(end 165.3325 95.0175)
@@
 	)
 	(segment
-		(start 166.77 94.33)
-		(end 166.27 93.83)
-		(width 0.3)
-		(layer "F.Cu")
-		(net "/Power/PHYPWRBJT")
-	)
-	(segment
 		(start 168.52 94.33)
-		(end 166.77 94.33)
+		(end 167.26 94.33)
 		(width 0.3)
 		(layer "F.Cu")
@@
 	)
 	(segment
-		(start 166.27 93.83)
+		(start 167.26 94.33)
 		(end 166.27 93.34)
 		(width 0.3)
@@
 	)
 	(segment
-		(start 175.77 101.5175)
-		(end 175.77 102.33)
+		(start 178.02 88.58)
+		(end 169.03 88.58)
 		(width 0.2)
 		(layer "F.Cu")
@@
 	)
 	(segment
-		(start 175.77 102.33)
-		(end 175.52 102.58)
+		(start 169.03 88.58)
+		(end 165.775 85.325)
 		(width 0.2)
 		(layer "F.Cu")
@@
 	)
 	(segment
-		(start 178.02 88.58)
-		(end 169.03 88.58)
+		(start 185.02 105.33)
+		(end 185.02 95.58)
 		(width 0.2)
 		(layer "F.Cu")
@@
 	)
 	(segment
-		(start 175.52 102.58)
-		(end 175.52 106.08)
+		(start 175.77 102.33)
+		(end 175.52 102.58)
 		(width 0.2)
 		(layer "F.Cu")
@@
 	)
 	(segment
-		(start 185.02 95.58)
-		(end 178.02 88.58)
+		(start 175.77 101.5175)
+		(end 175.77 102.33)
 		(width 0.2)
 		(layer "F.Cu")
@@
 	)
 	(segment
-		(start 169.03 88.58)
-		(end 165.775 85.325)
+		(start 185.02 95.58)
+		(end 178.02 88.58)
 		(width 0.2)
 		(layer "F.Cu")
@@
 	)
 	(segment
-		(start 181.77 106.83)
-		(end 185.02 103.58)
+		(start 175.52 106.08)
+		(end 176.27 106.83)
 		(width 0.2)
 		(layer "F.Cu")
@@
 	)
 	(segment
-		(start 175.52 106.08)
-		(end 176.27 106.83)
+		(start 176.27 106.83)
+		(end 183.52 106.83)
 		(width 0.2)
 		(layer "F.Cu")
@@
 	)
 	(segment
-		(start 176.27 106.83)
-		(end 181.77 106.83)
+		(start 175.52 102.58)
+		(end 175.52 106.08)
 		(width 0.2)
 		(layer "F.Cu")
@@
 	)
 	(segment
-		(start 185.02 103.58)
-		(end 185.02 95.58)
+		(start 183.52 106.83)
+		(end 185.02 105.33)
 		(width 0.2)
 		(layer "F.Cu")

Commit message: Update esp-24v-16ch-v6.kicad_pcb
Parts:
- L2: footprint Tales:L_12x12mm_h6mm -> Tales:L_12x12mm_H6mm
- moved C11 0.50 mm to (162.8, 96.1)
- moved C12 0.25 mm to (164.5, 95.6)
- moved L3 0.25 mm to (166.0, 96.1)
- moved Q1 0.25 mm to (160.0, 95.8)
- moved R8 0.25 mm to (159.5, 93.3)
Routing:
- net /MCU/PHYPWR: track 31.4 -> 30.1 mm
- net /OUTPUT16: track 44.5 -> 45.2 mm
- net /OUTPUT15: track 40.1 -> 40.8 mm
- net GND: track 144.3 -> 143.8 mm
