File: V6/esp-24v-16ch-v6.kicad_pcb (KiCad board)
At the start: 4 copper layers, 128 x 67.8 mm, 344 parts, among them J1 250-208, J2 250-202, J3 250-208, J4 250-208, J5 250-208, J6 250-202, J7 USB_C_Receptacle_USB2.0, J8 ETHERNET, J9 250-203, Q1 WPM2015-3/TR, Q10 MMBT2222A, Q11 MMBT2222A, Q12 MMBT2222A, Q13 MMBT2222A, Q14 MMBT2222A, Q15 MMBT2222A, Q16 MMBT2222A, Q17 MMBT2222A, Q18 MMBT2222A, Q19 MMBT2222A, Q2 MMUN2211LT3G, Q3 UMH3N, Q4 MMBT2222A, Q5 MMBT2222A, Q6 MMBT2222A, Q7 MMBT2222A, Q8 MMBT2222A, Q9 MMBT2222A, SW1 RESET, SW2 1WIRE_SEL, U1 SY8089A1AAC, U10 OR-3H7-4, U11 OR-3H7-4, U12 OR-3H7-4, U13 OR-3H7-4, U2 TX4138, U3 CH340K, U4 ESP32-WROOM-32UE-N16, U5 LAN8710A, U6 MCP23008, U7 MCP23008, U8 MCP23017, U9 DS2482S-100

Commit message: Added relase date to PCB
Other:
- board text added: "V6.0.2 2026-06-08"
Changed lines of the file:
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@@
 	)
 	(gr_rect
+		(start 155.77 130.08)
+		(end 161.27 132.83)
+		(stroke
+			(width 0.1)
+			(type solid)
+		)
+		(fill no)
+		(layer "F.SilkS")
+	)
+	(gr_rect
 		(start 187.77 98.08)
 		(end 215.77 99.83)
@@
 		(layer "Edge.Cuts")
 	)
+	(gr_text "V6.0.2\n2026-06-08"
+		(at 158.52 132.58 0)
+		(layer "F.SilkS")
+		(effects
+			(font
+				(size 0.8 0.5)
+				(thickness 0.1)
+			)
+			(justify bottom)
+		)
+	)
 	(gr_text "RESET"
 		(at 158.52 78.08 0)
@@
 	)
 	(segment
+		(start 144.52 82.91)
+		(end 145.19 82.91)
+		(width 0.3)
+		(layer "F.Cu")
+		(net "+5V")
+	)
+	(segment
+		(start 147.77 78.83)
+		(end 147.77 76.58)
+		(width 1.5)
+		(layer "F.Cu")
+		(net "+5V")
+	)
+	(segment
+		(start 147.26 82.88)
+		(end 147.29 82.85)
+		(width 0.5)
+		(layer "F.Cu")
+		(net "+5V")
+	)
+	(segment
+		(start 146.27 80.33)
+		(end 147.77 78.83)
+		(width 1)
+		(layer "F.Cu")
+		(net "+5V")
+	)
+	(segment
+		(start 148.02 82.85)
+		(end 147.29 82.85)
+		(width 0.5)
+		(layer "F.Cu")
+		(net "+5V")
+	)
+	(segment
+		(start 146.27 82.88)
+		(end 147.26 82.88)
+		(width 0.5)
+		(layer "F.Cu")
+		(net "+5V")
+	)
+	(segment
+		(start 146.27 82.88)
+		(end 145.22 82.88)
+		(width 0.3)
+		(layer "F.Cu")
+		(net "+5V")
+	)
+	(segment
+		(start 146.27 82.88)
+		(end 146.27 82.08)
+		(width 1)
+		(layer "F.Cu")
+		(net "+5V")
+	)
+	(segment
+		(start 149.32 94.38)
+		(end 149.32 93.58)
+		(width 0.5)
+		(layer "F.Cu")
+		(net "+5V")
+	)
+	(segment
+		(start 146.27 80.33)
+		(end 146.27 82.08)
+		(width 1)
+		(layer "F.Cu")
+		(net "+5V")
+	)
+	(segment
+		(start 145.22 82.88)
+		(end 145.19 82.91)
+		(width 0.3)
+		(layer "F.Cu")
+		(net "+5V")
+	)
+	(via
+		(at 146.27 80.33)
+		(size 0.6)
+		(drill 0.3)
+		(layers "F.Cu" "B.Cu")
+		(net "+5V")
+	)
+	(via
+		(at 154.77 96.33)
+		(size 0.6)
+		(drill 0.3)
+		(layers "F.Cu" "B.Cu")
+		(net "+5V")
+	)
+	(via
+		(at 153.02 96.33)
+		(size 0.6)
+		(drill 0.3)
+		(layers "F.Cu" "B.Cu")
+		(capping no)
+		(covering
+			(front no)
+			(back no)
+		)
+		(plugging
+			(front no)
+			(back no)
+		)
+		(filling no)
+		(net "+5V")
+	)
+	(via
+		(at 149.32 93.58)
+		(size 0.6)
+		(drill 0.3)
+		(layers "F.Cu" "B.Cu")
+		(capping no)
+		(covering
+			(front no)
+			(back no)
+		)
+		(plugging
+			(front no)
+			(back no)
+		)
+		(filling no)
+		(net "+5V")
+	)
+	(via
+		(at 146.27 82.08)
+		(size 0.6)
+		(drill 0.3)
+		(layers "F.Cu" "B.Cu")
+		(net "+5V")
+	)
+	(segment
+		(start 146.27 90.53)
+		(end 146.27 80.332)
+		(width 1)
+		(layer "B.Cu")
+		(net "+5V")
+	)
+	(segment
+		(start 149.32 93.58)
+		(end 150.27 93.58)
+		(width 1)
+		(layer "B.Cu")
+		(net "+5V")
+	)
+	(segment
+		(start 146.27 90.53)
+		(end 149.32 93.58)
+		(width 1)
+		(layer "B.Cu")
+		(net "+5V")
+	)
+	(segment
+		(start 150.27 93.58)
+		(end 153.02 96.33)
+		(width 1)
+		(layer "B.Cu")
+		(net "+5V")
+	)
+	(segment
+		(start 154.77 96.33)
+		(end 153.02 96.33)
+		(width 1)
+		(layer "B.Cu")
+		(net "+5V")
+	)
+	(segment
+		(start 168.02 109.58)
+		(end 165.77 109.58)
+		(width 0.5)
+		(layer "F.Cu")
+		(net "/Power/5VSH")
+	)
+	(segment
+		(start 165.52 109.33)
+		(end 165.52 106.33)
+		(width 0.5)
+		(layer "F.Cu")
+		(net "/Power/5VSH")
+	)
+	(segment
+		(start 165.52 100.83)
+		(end 165.495 100.805)
+		(width 1.2)
+		(layer "F.Cu")
+		(net "/Power/5VSH")
+	)
+	(segment
+		(start 165.52 102.58)
+		(end 165.52 100.83)
+		(width 1.2)
+		(layer "F.Cu")
+		(net "/Power/5VSH")
+	)
+	(segment
+		(start 165.52 106.33)
+		(end 165.52 102.58)
+		(width 1.5)
+		(layer "F.Cu")
+		(net "/Power/5VSH")
+	)
+	(segment
+		(start 165.495 100.805)
+		(end 165.495 99.33)
+		(width 1.2)
+		(layer "F.Cu")
+		(net "/Power/5VSH")
+	)
+	(segment
+		(start 165.77 109.58)
+		(end 165.52 109.33)
+		(width 0.5)
+		(layer "F.Cu")
+		(net "/Power/5VSH")
+	)
+	(segment
 		(start 179.775 95.08)
 		(end 178.52 96.335)
@@
 	)
 	(segment
-		(start 144.52 82.91)
-		(end 145.19 82.91)
-		(width 0.3)
-		(layer "F.Cu")
-		(net "+5V")
-	)
-	(segment
-		(start 147.77 78.83)
-		(end 147.77 76.58)
-		(width 1.5)
-		(layer "F.Cu")
-		(net "+5V")
-	)
-	(segment
-		(start 147.26 82.88)
-		(end 147.29 82.85)
-		(width 0.5)
-		(layer "F.Cu")
-		(net "+5V")
-	)
-	(segment
-		(start 146.27 80.33)
-		(end 147.77 78.83)
-		(width 1)
-		(layer "F.Cu")
-		(net "+5V")
-	)
-	(segment
-		(start 148.02 82.85)
-		(end 147.29 82.85)
-		(width 0.5)
-		(layer "F.Cu")
-		(net "+5V")
-	)
-	(segment
-		(start 146.27 82.88)
-		(end 147.26 82.88)
-		(width 0.5)
-		(layer "F.Cu")
-		(net "+5V")
-	)
-	(segment
-		(start 146.27 82.88)
-		(end 145.22 82.88)
-		(width 0.3)
-		(layer "F.Cu")
-		(net "+5V")
-	)
-	(segment
-		(start 146.27 82.88)
-		(end 146.27 82.08)
-		(width 1)
-		(layer "F.Cu")
-		(net "+5V")
-	)
-	(segment
-		(start 149.32 94.38)
-		(end 149.32 93.58)
-		(width 0.5)
-		(layer "F.Cu")
-		(net "+5V")
-	)
-	(segment
-		(start 146.27 80.33)
-		(end 146.27 82.08)
-		(width 1)
-		(layer "F.Cu")
-		(net "+5V")
-	)
-	(segment
-		(start 145.22 82.88)
-		(end 145.19 82.91)
-		(width 0.3)
-		(layer "F.Cu")
-		(net "+5V")
-	)
-	(via
-		(at 146.27 80.33)
-		(size 0.6)
-		(drill 0.3)
-		(layers "F.Cu" "B.Cu")
-		(net "+5V")
-	)
-	(via
-		(at 154.77 96.33)
-		(size 0.6)
-		(drill 0.3)
-		(layers "F.Cu" "B.Cu")
-		(net "+5V")
-	)
-	(via
-		(at 153.02 96.33)
-		(size 0.6)
-		(drill 0.3)
-		(layers "F.Cu" "B.Cu")
-		(capping no)
-		(covering
-			(front no)
-			(back no)
-		)
-		(plugging
-			(front no)
-			(back no)
-		)
-		(filling no)
-		(net "+5V")
-	)
-	(via
-		(at 149.32 93.58)
-		(size 0.6)
-		(drill 0.3)
-		(layers "F.Cu" "B.Cu")
-		(capping no)
-		(covering
-			(front no)
-			(back no)
-		)
-		(plugging
-			(front no)
-			(back no)
-		)
-		(filling no)
-		(net "+5V")
-	)
-	(via
-		(at 146.27 82.08)
-		(size 0.6)
-		(drill 0.3)
-		(layers "F.Cu" "B.Cu")
-		(net "+5V")
-	)
-	(segment
-		(start 146.27 90.53)
-		(end 146.27 80.332)
-		(width 1)
-		(layer "B.Cu")
-		(net "+5V")
-	)
-	(segment
-		(start 149.32 93.58)
-		(end 150.27 93.58)
-		(width 1)
-		(layer "B.Cu")
-		(net "+5V")
-	)
-	(segment
-		(start 146.27 90.53)
-		(end 149.32 93.58)
-		(width 1)
-		(layer "B.Cu")
-		(net "+5V")
-	)
-	(segment
-		(start 150.27 93.58)
-		(end 153.02 96.33)
-		(width 1)
-		(layer "B.Cu")
-		(net "+5V")
-	)
-	(segment
-		(start 154.77 96.33)
-		(end 153.02 96.33)
-		(width 1)
-		(layer "B.Cu")
-		(net "+5V")
-	)
-	(segment
 		(start 199.2325 113.7925)
 		(end 199.195 113.755)
@@
 		(net "/Output 11/OUTBASE")
 	)
-	(segment
-		(start 168.02 109.58)
-		(end 165.77 109.58)
-		(width 0.5)
-		(layer "F.Cu")
-		(net "/Power/5VSH")
-	)
-	(segment
-		(start 165.52 109.33)
-		(end 165.52 106.33)
-		(width 0.5)
-		(layer "F.Cu")
-		(net "/Power/5VSH")
-	)
-	(segment
-		(start 165.52 100.83)
-		(end 165.495 100.805)
-		(width 1.2)
-		(layer "F.Cu")
-		(net "/Power/5VSH")
-	)
-	(segment
-		(start 165.52 102.58)
-		(end 165.52 100.83)
-		(width 1.2)
-		(layer "F.Cu")
-		(net "/Power/5VSH")
-	)
-	(segment
-		(start 165.52 106.33)
-		(end 165.52 102.58)
-		(width 1.5)
-		(layer "F.Cu")
-		(net "/Power/5VSH")
-	)
-	(segment
-		(start 165.495 100.805)
-		(end 165.495 99.33)
-		(width 1.2)
-		(layer "F.Cu")
-		(net "/Power/5VSH")
-	)
-	(segment
-		(start 165.77 109.58)
-		(end 165.52 109.33)
-		(width 0.5)
-		(layer "F.Cu")
-		(net "/Power/5VSH")
-	)
 	(zone

Commit message: Cleanup
Parts:
- R20: value 10k -> 1.5k
Changed lines of the file:
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@@
 			(unit
 				(name "A")
-				(pins "3" "4" "5" "21" "22" "17" "18" "20" "19" "32" "2" "1" "38" "39"
-					"15" "25" "35" "24" "34" "26" "29" "14" "16" "13" "23" "27" "28" "30"
+				(pins "3" "4" "5" "21" "22" "17" "18" "20" "19" "32" "2" "1" "38" "15"
+					"39" "25" "35" "24" "34" "26" "29" "14" "16" "13" "23" "27" "28" "30"
 					"31" "33" "36" "37" "10" "11" "12" "8" "9" "6" "7"
 				)
@@
 		(tags "resistor")
 		(property "Reference" "R23"
-			(at -2.5 0 180)
+			(at 2 0 180)
 			(layer "F.SilkS")
 			(effects
@@
 		(tags "capacitor")
 		(property "Reference" "C23"
-			(at 2.5 0 180)
+			(at -2 0 180)
 			(layer "F.SilkS")
 			(effects
@@
 		(tags "resistor")
 		(property "Reference" "R20"
-			(at -1.5 0.25 180)
+			(at -1.5 0 180)
 			(layer "F.SilkS")
 			(effects
@@
 			)
 		)
-		(property "Value" "10k"
+		(property "Value" "1.5k"
 			(at 0 1.17 90)
 			(layer "F.Fab")
@@
 			)
 		)
-		(property "Mfr PN" "0402WGF1002TCE"
+		(property "Mfr PN" "0402WGF1501TCE"
 			(at 0 0 270)
 			(unlocked yes)
@@
 			)
 		)
-		(property "Vendor PN" "C25744"
+		(property "Vendor PN" "C25867"
 			(at 0 0 270)
 			(unlocked yes)
@@
 			)
 		)
-		(property "LCSC Part #" "C25744"
+		(property "LCSC Part #" "C25867"
 			(at 0 0 270)
 			(unlocked yes)
@@
 		(tags "resistor")
 		(property "Reference" "R25"
-			(at -2.5 0 180)
+			(at 2 0 180)
 			(layer "F.SilkS")
 			(effects

Commit message: Update resistance value for pull-ups.
Parts:
- R21, R23, R25, R26, R27, R28, R29: value 10k -> 2.2k
Changed lines of the file:
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@@
 			)
 		)
-		(property "Value" "10k"
+		(property "Value" "2.2k"
 			(at 0 1.17 90)
 			(layer "F.Fab")
@@
 			)
 		)
-		(property "Mfr PN" "0402WGF1002TCE"
+		(property "Mfr PN" "0402WGF2201TCE"
 			(at 0 0 270)
 			(unlocked yes)
@@
 			)
 		)
-		(property "LCSC Part #" "C25744"
+		(property "LCSC Part #" "C25879"
 			(at 0 0 270)
 			(unlocked yes)
@@
 			)
 		)
-		(property "Value" "10k"
+		(property "Value" "2.2k"
 			(at 0 1.17 90)
 			(layer "F.Fab")
@@
 			)
 		)
-		(property "Mfr PN" "0402WGF1002TCE"
+		(property "Mfr PN" "0402WGF2201TCE"
 			(at 0 0 270)
 			(unlocked yes)
@@
 			)
 		)
-		(property "LCSC Part #" "C25744"
+		(property "LCSC Part #" "C25879"
 			(at 0 0 270)
 			(unlocked yes)
@@
 			)
 		)
-		(property "Value" "10k"
+		(property "Value" "2.2k"
 			(at 0 1.17 90)
 			(layer "F.Fab")
@@
 			)
 		)
-		(property "Mfr PN" "0402WGF1002TCE"
+		(property "Mfr PN" "0402WGF2201TCE"
 			(at 0 0 270)
 			(unlocked yes)
@@
 			)
 		)
-		(property "LCSC Part #" "C25744"
+		(property "LCSC Part #" "C25879"
 			(at 0 0 270)
 			(unlocked yes)
@@
 			)
 		)
-		(property "Value" "10k"
+		(property "Value" "2.2k"
 			(at 0 1.17 90)
 			(layer "F.Fab")
@@
 			)
 		)
-		(property "Mfr PN" "0402WGF1002TCE"
+		(property "Mfr PN" "0402WGF2201TCE"
 			(at 0 0 270)
 			(unlocked yes)
@@
 			)
 		)
-		(property "LCSC Part #" "C25744"
+		(property "LCSC Part #" "C25879"
 			(at 0 0 270)
 			(unlocked yes)
@@
 			)
 		)
-		(property "Value" "10k"
+		(property "Value" "2.2k"
 			(at 0 1.17 90)
 			(layer "F.Fab")
@@
 			)
 		)
-		(property "Mfr PN" "0402WGF1002TCE"
+		(property "Mfr PN" "0402WGF2201TCE"
 			(at 0 0 270)
 			(unlocked yes)
@@
 			)
 		)
-		(property "Vendor PN" "C25744"
+		(property "Vendor PN" "C25879"
 			(at 0 0 270)
 			(unlocked yes)
@@
 			)
 		)
-		(property "LCSC Part #" "C25744"
+		(property "LCSC Part #" "C25879"
 			(at 0 0 270)
 			(unlocked yes)
@@
 			)
 		)
-		(property "Value" "10k"
+		(property "Value" "2.2k"
 			(at 0 1.17 90)
 			(layer "F.Fab")
@@
 			)
 		)
-		(property "Mfr PN" "0402WGF1002TCE"
+		(property "Mfr PN" "0402WGF2201TCE"
 			(at 0 0 270)
 			(unlocked yes)
@@
 			)
 		)
-		(property "LCSC Part #" "C25744"
+		(property "LCSC Part #" "C25879"
 			(at 0 0 270)
 			(unlocked yes)
@@
 			)
 		)
-		(property "Value" "10k"
+		(property "Value" "2.2k"
 			(at 0 1.17 90)
 			(layer "F.Fab")
@@
 			)
 		)
-		(property "Mfr PN" "0402WGF1002TCE"
+		(property "Mfr PN" "0402WGF2201TCE"
 			(at 0 0 270)
 			(unlocked yes)
@@
 			)
 		)
-		(property "LCSC Part #" "C25744"
+		(property "LCSC Part #" "C25879"
 			(at 0 0 270)
 			(unlocked yes)
