File: V6/esp-24v-16ch-v6-inputs9-16.kicad_sch (KiCad schematic)
At the start: 10 parts, among them U11 OR-3H7-4

Commit message: V6 is up
Parts:
- renumbered C46 to C54, C47 to C55, D33 to D34, D34 to D35, D35 to D36, R64 to R65, R65 to R66, R66 to R67, U11 to U12
Connections:
- net GND: now also U12.9; no longer C54.2, C55.2, D34.2 (A2), D35.1 (K), U12.15, U12.2
- net INOPTO: now also U12.7; no longer U12.1
- net MUXIN: now also U12.10; no longer U12.16
- new net GNDIO: C54.2, C55.2, D34.2 (A2), D35.1 (K), U12.8

Commit message: Revising power rails
Parts:
- renumbered C54 to C55, C55 to C56

Commit message: Added voltage monitors for both ESP32 and LAN8710A
Parts:
- renumbered C55 to C53, C56 to C54, D36 to D34, D34 to D35, D35 to D36, R67 to R65, R65 to R67, U12 to U14
