File: V6/esp-24v-16ch-v6-mcu.kicad_sch (KiCad schematic)
At the start: 17 parts, among them Q3 UMH3N, SW1 RESET, U3 CH340K, U4 ESP32-WROOM-32UE-N16

Commit message: V6 is up
Parts:
- removed R15: 2k2, Tales:R_0402_1005Metric, symbol Device:R_US
- added R16: 2k2, Tales:R_0402_1005Metric, symbol Device:R_US
- C13, C16: value 10uF/10V -> 10uF/25V; footprint Tales:C_0603_1608Metric -> Tales:C_0805_2012Metric; Case 0603/1608 -> 0805/2012; LCSC Part # C19702 -> C15850; Mfr PN CL10A106KP8NNNC -> CL21A106KAYNNNE; Vendor PN C19702 -> C15850
- C14, C15, R12, R13: Package 0402/1005 -> (none)
- R18: renamed from R16; Package 0402/1005 -> (none)
- renumbered R17 to R14, R14 to R15, R18 to R17
Connections:
- net +3V3: now also R16.1
- net INPUT1: no longer names the net of U4.6 (IO34)
- net INPUT2: no longer names the net of U4.7 (IO35)
- net MCPININTA renamed MCPIN1INT
- net MCPININTB renamed MCPIN2INT
- net MCPIN2INT: now also R16.2
- no-connect marks 13 -> 15
Other:
- note added: "TEMPLATE FOR GPIO ASSIGNMENT {"NAME":"ESP-24V-16CH-V6","GPIO":[0,3200,0,3232,0,0,0,0,5536,10240,10241,0,0, 0,5600,0,0,0,0,5568,0,0,0,0,0,0,0,0,608,640,192,193,0,0,0,0],"FLAG":0,"BASE":1} See https://tasmota.github.io/docs/Templates/"
- note added: "TEMPLATE FOR MCP23017 I/O ASSIGNMENT {"NAME":"MCP23017 expander","BASE":0,"GPIO":[192,193,194,195,196,197,198,0,199,200,201, 202,203,204,205,0,224,225,226,227,228,229,230,231,232,233,234,235,236,237,238,239], "IOCON":0x5C} Save as mcp23x.dat and load into tasmota's filesystem. See https://tasmota.github.io/docs/MCP230xx/"
- note removed: "TEMPLATE FOR GPIO ASSIGNMENT {"NAME":"ESP-24V-16CH-V5","GPIO":[0,3200,0,3232,0,0,0,0,5536,10240,10241,0,0, 0,5600,0,0,0,0,5568,0,0,0,0,0,0,0,0,608,640,192,193,0,0,0,0],"FLAG":0,"BASE":1} See https://tasmota.github.io/docs/Templates/"
- note removed: "TEMPLATE FOR MCP23017 I/O ASSIGNMENT {"NAME":"MCP23017 expander","BASE":0,"GPIO":[192,193,194,195,196,197,198,0,199,200,201, 202,203,204,205,0,224,225,226,227,228,229,230,231,232,233,234,235,236,237,238,239]} Save as mcp23x.dat and load into tasmota's filesystem. See https://tasmota.github.io/docs/MCP230xx/"

Commit message: Revising power rails
Parts:
- renumbered C13 to C15, C14 to C16, C15 to C17, C16 to C18, C17 to C19
Changed lines of the file:
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@@
 		(in_pos_files yes)
 		(dnp no)
-		(property "Reference" "#PWR046"
+		(property "Reference" "#PWR048"
 			(at 260.35 107.95 0)
 			(hide yes)
@@
 			(project "esp-24v-16ch-v6"
 				(path "/2bc5a21a-1d79-419d-a592-6852cc07b00a/f2a42251-1da5-495a-abaf-29698c5bb0fe"
-					(reference "#PWR046")
+					(reference "#PWR048")
 					(unit 1)
 				)
@@
 		(in_pos_files yes)
 		(dnp no)
-		(property "Reference" "C16"
+		(property "Reference" "C18"
 			(at 162.56 50.8 0)
 			(show_name no)
@@
 			(project "esp-24v-16ch-v6"
 				(path "/2bc5a21a-1d79-419d-a592-6852cc07b00a/f2a42251-1da5-495a-abaf-29698c5bb0fe"
-					(reference "C16")
+					(reference "C18")
 					(unit 1)
 				)
@@
 		(in_pos_files yes)
 		(dnp no)
-		(property "Reference" "C17"
+		(property "Reference" "C19"
 			(at 185.42 50.8 0)
 			(show_name no)
@@
 			(project "esp-24v-16ch-v6"
 				(path "/2bc5a21a-1d79-419d-a592-6852cc07b00a/f2a42251-1da5-495a-abaf-29698c5bb0fe"
-					(reference "C17")
+					(reference "C19")
 					(unit 1)
 				)
@@
 		(dnp no)
 		(fields_autoplaced yes)
-		(property "Reference" "#PWR040"
+		(property "Reference" "#PWR042"
 			(at 182.88 63.5 0)
 			(hide yes)
@@
 			(project "esp-24v-16ch-v6"
 				(path "/2bc5a21a-1d79-419d-a592-6852cc07b00a/f2a42251-1da5-495a-abaf-29698c5bb0fe"
-					(reference "#PWR040")
+					(reference "#PWR042")
 					(unit 1)
 				)
@@
 		(dnp no)
 		(fields_autoplaced yes)
-		(property "Reference" "#PWR031"
+		(property "Reference" "#PWR033"
 			(at 43.18 59.69 0)
 			(hide yes)
@@
 			(project "esp-24v-16ch-v6"
 				(path "/2bc5a21a-1d79-419d-a592-6852cc07b00a/f2a42251-1da5-495a-abaf-29698c5bb0fe"
-					(reference "#PWR031")
+					(reference "#PWR033")
 					(unit 1)
 				)
@@
 		(dnp no)
 		(fields_autoplaced yes)
-		(property "Reference" "#PWR037"
+		(property "Reference" "#PWR039"
 			(at 160.02 63.5 0)
 			(hide yes)
@@
 			(project "esp-24v-16ch-v6"
 				(path "/2bc5a21a-1d79-419d-a592-6852cc07b00a/f2a42251-1da5-495a-abaf-29698c5bb0fe"
-					(reference "#PWR037")
+					(reference "#PWR039")
 					(unit 1)
 				)
@@
 		(dnp no)
 		(fields_autoplaced yes)
-		(property "Reference" "#PWR045"
+		(property "Reference" "#PWR047"
 			(at 257.81 99.06 0)
 			(hide yes)
@@
 			(project "esp-24v-16ch-v6"
 				(path "/2bc5a21a-1d79-419d-a592-6852cc07b00a/f2a42251-1da5-495a-abaf-29698c5bb0fe"
-					(reference "#PWR045")
+					(reference "#PWR047")
 					(unit 1)
 				)
@@
 		(dnp no)
 		(fields_autoplaced yes)
-		(property "Reference" "#PWR030"
+		(property "Reference" "#PWR032"
 			(at 21.59 59.69 0)
 			(hide yes)
@@
 			(project "esp-24v-16ch-v6"
 				(path "/2bc5a21a-1d79-419d-a592-6852cc07b00a/f2a42251-1da5-495a-abaf-29698c5bb0fe"
-					(reference "#PWR030")
+					(reference "#PWR032")
 					(unit 1)
 				)
@@
 		(dnp no)
 		(fields_autoplaced yes)
-		(property "Reference" "C13"
+		(property "Reference" "C15"
 			(at 24.13 44.4562 0)
 			(show_name no)
@@
 			(project "esp-24v-16ch-v6"
 				(path "/2bc5a21a-1d79-419d-a592-6852cc07b00a/f2a42251-1da5-495a-abaf-29698c5bb0fe"
-					(reference "C13")
+					(reference "C15")
 					(unit 1)
 				)
@@
 		(in_pos_files yes)
 		(dnp no)
-		(property "Reference" "#PWR032"
+		(property "Reference" "#PWR034"
 			(at 63.5 41.91 0)
 			(hide yes)
@@
 			(project "esp-24v-16ch-v6"
 				(path "/2bc5a21a-1d79-419d-a592-6852cc07b00a/f2a42251-1da5-495a-abaf-29698c5bb0fe"
-					(reference "#PWR032")
+					(reference "#PWR034")
 					(unit 1)
 				)
@@
 		(in_pos_files yes)
 		(dnp no)
-		(property "Reference" "#PWR035"
+		(property "Reference" "#PWR037"
 			(at 140.97 55.88 0)
 			(hide yes)
@@
 			(project "esp-24v-16ch-v6"
 				(path "/2bc5a21a-1d79-419d-a592-6852cc07b00a/f2a42251-1da5-495a-abaf-29698c5bb0fe"
-					(reference "#PWR035")
+					(reference "#PWR037")
 					(unit 1)
 				)
@@
 		(dnp no)
 		(fields_autoplaced yes)
-		(property "Reference" "#PWR033"
+		(property "Reference" "#PWR035"
 			(at 63.5 95.25 0)
 			(hide yes)
@@
 			(project "esp-24v-16ch-v6"
 				(path "/2bc5a21a-1d79-419d-a592-6852cc07b00a/f2a42251-1da5-495a-abaf-29698c5bb0fe"
-					(reference "#PWR033")
+					(reference "#PWR035")
 					(unit 1)
 				)
@@
 		(dnp no)
 		(fields_autoplaced yes)
-		(property "Reference" "C15"
+		(property "Reference" "C17"
 			(at 143.51 68.5862 0)
 			(show_name no)
@@
 			(project "esp-24v-16ch-v6"
 				(path "/2bc5a21a-1d79-419d-a592-6852cc07b00a/f2a42251-1da5-495a-abaf-29698c5bb0fe"
-					(reference "C15")
+					(reference "C17")
 					(unit 1)
 				)
@@
 		(in_pos_files yes)
 		(dnp no)
-		(property "Reference" "#PWR038"
+		(property "Reference" "#PWR040"
 			(at 179.07 50.8 0)
 			(hide yes)
@@
 			(project "esp-24v-16ch-v6"
 				(path "/2bc5a21a-1d79-419d-a592-6852cc07b00a/f2a42251-1da5-495a-abaf-29698c5bb0fe"
-					(reference "#PWR038")
+					(reference "#PWR040")
 					(unit 1)
 				)
@@
 		(dnp no)
 		(fields_autoplaced yes)
-		(property "Reference" "#PWR034"
+		(property "Reference" "#PWR036"
 			(at 128.27 110.49 0)
 			(hide yes)
@@
 			(project "esp-24v-16ch-v6"
 				(path "/2bc5a21a-1d79-419d-a592-6852cc07b00a/f2a42251-1da5-495a-abaf-29698c5bb0fe"
-					(reference "#PWR034")
+					(reference "#PWR036")
 					(unit 1)
 				)
@@
 		(in_pos_files yes)
 		(dnp no)
-		(property "Reference" "#PWR043"
+		(property "Reference" "#PWR045"
 			(at 245.11 59.69 0)
 			(hide yes)
@@
 			(project "esp-24v-16ch-v6"
 				(path "/2bc5a21a-1d79-419d-a592-6852cc07b00a/f2a42251-1da5-495a-abaf-29698c5bb0fe"
-					(reference "#PWR043")
+					(reference "#PWR045")
 					(unit 1)
 				)
@@
 		(in_pos_files yes)
 		(dnp no)
-		(property "Reference" "#PWR042"
+		(property "Reference" "#PWR044"
 			(at 232.41 59.69 0)
 			(hide yes)
@@
 			(project "esp-24v-16ch-v6"
 				(path "/2bc5a21a-1d79-419d-a592-6852cc07b00a/f2a42251-1da5-495a-abaf-29698c5bb0fe"
-					(reference "#PWR042")
+					(reference "#PWR044")
 					(unit 1)
 				)
@@
 		(dnp no)
 		(fields_autoplaced yes)
-		(property "Reference" "#PWR036"
+		(property "Reference" "#PWR038"
 			(at 140.97 83.82 0)
 			(hide yes)
@@
 			(project "esp-24v-16ch-v6"
 				(path "/2bc5a21a-1d79-419d-a592-6852cc07b00a/f2a42251-1da5-495a-abaf-29698c5bb0fe"
-					(reference "#PWR036")
+					(reference "#PWR038")
 					(unit 1)
 				)
@@
 		(dnp no)
 		(fields_autoplaced yes)
-		(property "Reference" "#PWR039"
+		(property "Reference" "#PWR041"
 			(at 179.07 139.7 0)
 			(hide yes)
@@
 			(project "esp-24v-16ch-v6"
 				(path "/2bc5a21a-1d79-419d-a592-6852cc07b00a/f2a42251-1da5-495a-abaf-29698c5bb0fe"
-					(reference "#PWR039")
+					(reference "#PWR041")
 					(unit 1)
 				)
@@
 		(dnp no)
 		(fields_autoplaced yes)
-		(property "Reference" "C14"
+		(property "Reference" "C16"
 			(at 45.72 44.4562 0)
 			(show_name no)
@@
 			(project "esp-24v-16ch-v6"
 				(path "/2bc5a21a-1d79-419d-a592-6852cc07b00a/f2a42251-1da5-495a-abaf-29698c5bb0fe"
-					(reference "C14")
+					(reference "C16")
 					(unit 1)
 				)
@@
 		(in_pos_files yes)
 		(dnp no)
-		(property "Reference" "#PWR041"
+		(property "Reference" "#PWR043"
 			(at 209.55 55.88 0)
 			(hide yes)
@@
 			(project "esp-24v-16ch-v6"
 				(path "/2bc5a21a-1d79-419d-a592-6852cc07b00a/f2a42251-1da5-495a-abaf-29698c5bb0fe"
-					(reference "#PWR041")
+					(reference "#PWR043")
 					(unit 1)
 				)
@@
 		(in_pos_files yes)
 		(dnp no)
-		(property "Reference" "#PWR044"
+		(property "Reference" "#PWR046"
 			(at 246.38 107.95 0)
 			(hide yes)
@@
 			(project "esp-24v-16ch-v6"
 				(path "/2bc5a21a-1d79-419d-a592-6852cc07b00a/f2a42251-1da5-495a-abaf-29698c5bb0fe"
-					(reference "#PWR044")
+					(reference "#PWR046")
 					(unit 1)
 				)

Commit message: Included test points
Parts:
- added TP10: D+, TestPoint:TestPoint_Pad_D1.5mm, symbol Connector:TestPoint
- added TP11: D-, TestPoint:TestPoint_Pad_D1.5mm, symbol Connector:TestPoint
- added TP12: ESPEN, TestPoint:TestPoint_Pad_D1.5mm, symbol Connector:TestPoint
Connections:
- net ESPEN: now also TP12.1
- net USBD+: now also TP10.1
- net USBD-: now also TP11.1

Commit message: Included a shunt resistor on the 5V rail, for measuring current during development.
Parts:
- renumbered TP10 to TP11, TP11 to TP12, TP12 to TP13
Changed lines of the file:
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@@
 		(in_pos_files yes)
 		(dnp no)
-		(property "Reference" "TP10"
+		(property "Reference" "TP11"
 			(at 38.1 58.42 0)
 			(show_name no)
@@
 			(project "esp-24v-16ch-v6"
 				(path "/2bc5a21a-1d79-419d-a592-6852cc07b00a/f2a42251-1da5-495a-abaf-29698c5bb0fe"
-					(reference "TP10")
+					(reference "TP11")
 					(unit 1)
 				)
@@
 		(in_pos_files yes)
 		(dnp no)
-		(property "Reference" "TP11"
+		(property "Reference" "TP12"
 			(at 46.99 58.42 0)
 			(show_name no)
@@
 			(project "esp-24v-16ch-v6"
 				(path "/2bc5a21a-1d79-419d-a592-6852cc07b00a/f2a42251-1da5-495a-abaf-29698c5bb0fe"
-					(reference "TP11")
+					(reference "TP12")
 					(unit 1)
 				)
@@
 		(in_pos_files yes)
 		(dnp no)
-		(property "Reference" "TP12"
+		(property "Reference" "TP13"
 			(at 127 53.34 0)
 			(show_name no)
@@
 			(project "esp-24v-16ch-v6"
 				(path "/2bc5a21a-1d79-419d-a592-6852cc07b00a/f2a42251-1da5-495a-abaf-29698c5bb0fe"
-					(reference "TP12")
+					(reference "TP13")
 					(unit 1)
 				)

Commit message: Update resistance value for pull-ups.
Other:
- note added: "FOR NEXT VERSION: REPLACE THE RC RESET CIRCUIT FOR A TPS3820-33 (25ms)"
Changed lines of the file:
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@@
+		)
+	)
+	(text "FOR NEXT VERSION:\n REPLACE THE RC RESET CIRCUIT\n FOR A TPS3820-33 (25ms)"
+		(exclude_from_sim no)
+		(at 168.91 147.32 0)
+		(effects
+			(font
+				(size 1.905 1.905)
+			)
+			(justify left)
 		)
 	)

Commit message: Added voltage monitors for both ESP32 and LAN8710A
Parts:
- removed C17: 1uF/50V, Tales:C_0805_2012Metric, symbol Device:C_Small
- removed TP13: ESPEN, TestPoint:TestPoint_Pad_D1.5mm, symbol Connector:TestPoint
- added U3: TPS3820-33, Package_TO_SOT_SMD:SOT-23-5, symbol Power_Supervisor:TPS3823-xxDBV
- renumbered C18 to C17, C19 to C18, R12 to R13, R13 to R14, R18 to R17, R14 to R18, R17 to R19, R19 to R20, U3 to U4, U4 to U5
Connections:
- net +3V3: now also U3.5 (V_{DD})
- net ESPEN: now also U3.1 (~{RESET}); no longer Q3.6 (C1), R13.2, SW1.2
- net GND: now also U3.2 (GND)
- new net MRESET: Q3.6 (C1), R13.2, SW1.2, U3.3 (~{MR})
- no-connect marks 15 -> 16
Other:
- note added: "25ms RESET DELAY"
- note removed: "FOR NEXT VERSION: REPLACE THE RC RESET CIRCUIT FOR A TPS3820-33 (25ms)"
- moved on the sheet: R13, SW1
