File: V6/esp-24v-16ch-v6.kicad_sch (KiCad schematic)
At the start: 7 parts, among them J5 DB141V-2.54-8P, J6 DB141V-2.54-8P, J7 DB141V-2.54-8P, J8 DB141V-2.54-8P

Commit message: V6 is up
Parts:
- added FID4: Fiducial, Fiducial:Fiducial_1mm_Mask2mm, symbol Mechanical:Fiducial
- added J2: GNDIO, Tales:TerminalBlock_Wago_250-202_1x02_P3.5mm_45Degree, symbol Connector_Generic:Conn_01x02
- J1: renamed from J5; value DB141V-2.54-8P -> ENTRADAS 1-8; footprint Tales:TerminalBlock_Dibo_DB141V-2.54-8P_1x08_P2.54mm_Vertical -> Tales:TerminalBlock_Wago_250-208_1x08_P3.5mm_45Degree; LCSC Part # C2898750 -> C2833587; Mfr DIBO -> Wago; Mfr PN DB141V-2.54-8P -> 250-208; Vendor PN C2898750 -> C2833587
- J3: renamed from J6; value DB141V-2.54-8P -> ENTRADAS 9-16; footprint Tales:TerminalBlock_Dibo_DB141V-2.54-8P_1x08_P2.54mm_Vertical -> Tales:TerminalBlock_Wago_250-208_1x08_P3.5mm_45Degree; LCSC Part # C2898750 -> C2833587; Mfr DIBO -> Wago; Mfr PN DB141V-2.54-8P -> 250-208; Vendor PN C2898750 -> C2833587
- J4: renamed from J7; value DB141V-2.54-8P -> SAÍDAS 1-8; footprint Tales:TerminalBlock_Dibo_DB141V-2.54-8P_1x08_P2.54mm_Vertical -> Tales:TerminalBlock_Wago_250-208_1x08_P3.5mm_45Degree; LCSC Part # C2898750 -> C2833587; Mfr DIBO -> Wago; Mfr PN DB141V-2.54-8P -> 250-208; Vendor PN C2898750 -> C2833587
- J5: renamed from J8; value DB141V-2.54-8P -> SAÍDAS 9-16; footprint Tales:TerminalBlock_Dibo_DB141V-2.54-8P_1x08_P2.54mm_Vertical -> Tales:TerminalBlock_Wago_250-208_1x08_P3.5mm_45Degree; LCSC Part # C2898750 -> C2833587; Mfr DIBO -> Wago; Mfr PN DB141V-2.54-8P -> 250-208; Vendor PN C2898750 -> C2833587
Connections:
- new net GNDIO: J2.1 (Pin_1), J2.2 (Pin_2)
Other:
- sheet I2C Devices: file esp-24v-16ch-v5-i2c.kicad_sch -> esp-24v-16ch-v6-i2c.kicad_sch
- sheet I2C Devices ports: added IN1, IN2, MCPIN1INT, MCPIN2INT; removed MCPININTA, MCPININTB
- sheet Input 1: file esp-24v-16ch-v5-inputs1-8.kicad_sch -> esp-24v-16ch-v6-inputs1-8.kicad_sch
- sheet Input 10: file esp-24v-16ch-v5-inputs9-16.kicad_sch -> esp-24v-16ch-v6-inputs9-16.kicad_sch
- sheet Input 11: file esp-24v-16ch-v5-inputs9-16.kicad_sch -> esp-24v-16ch-v6-inputs9-16.kicad_sch
- sheet Input 12: file esp-24v-16ch-v5-inputs9-16.kicad_sch -> esp-24v-16ch-v6-inputs9-16.kicad_sch
- sheet Input 13: file esp-24v-16ch-v5-inputs9-16.kicad_sch -> esp-24v-16ch-v6-inputs9-16.kicad_sch
- sheet Input 14: file esp-24v-16ch-v5-inputs9-16.kicad_sch -> esp-24v-16ch-v6-inputs9-16.kicad_sch
- sheet Input 15: file esp-24v-16ch-v5-inputs9-16.kicad_sch -> esp-24v-16ch-v6-inputs9-16.kicad_sch
- sheet Input 16: file esp-24v-16ch-v5-inputs9-16.kicad_sch -> esp-24v-16ch-v6-inputs9-16.kicad_sch
- sheet Input 2: file esp-24v-16ch-v5-inputs1-8.kicad_sch -> esp-24v-16ch-v6-inputs1-8.kicad_sch
- sheet Input 3: file esp-24v-16ch-v5-inputs1-8.kicad_sch -> esp-24v-16ch-v6-inputs1-8.kicad_sch
- sheet Input 4: file esp-24v-16ch-v5-inputs1-8.kicad_sch -> esp-24v-16ch-v6-inputs1-8.kicad_sch
- sheet Input 5: file esp-24v-16ch-v5-inputs1-8.kicad_sch -> esp-24v-16ch-v6-inputs1-8.kicad_sch
- sheet Input 6: file esp-24v-16ch-v5-inputs1-8.kicad_sch -> esp-24v-16ch-v6-inputs1-8.kicad_sch
- sheet Input 7: file esp-24v-16ch-v5-inputs1-8.kicad_sch -> esp-24v-16ch-v6-inputs1-8.kicad_sch
- sheet Input 8: file esp-24v-16ch-v5-inputs1-8.kicad_sch -> esp-24v-16ch-v6-inputs1-8.kicad_sch
- sheet Input 9: file esp-24v-16ch-v5-inputs9-16.kicad_sch -> esp-24v-16ch-v6-inputs9-16.kicad_sch
- sheet LAN: file esp-24v-16ch-v5-lan.kicad_sch -> esp-24v-16ch-v6-lan.kicad_sch
- sheet MCU: file esp-24v-16ch-v5-mcu.kicad_sch -> esp-24v-16ch-v6-mcu.kicad_sch
- sheet MCU ports: added MCPIN1INT, MCPIN2INT; removed INPUT1, INPUT2, MCPININTA, MCPININTB
- sheet Output 1: file esp-24v-16ch-v5-outputs1-8.kicad_sch -> esp-24v-16ch-v6-outputs1-8.kicad_sch
- sheet Output 10: file esp-24v-16ch-v5-outputs9-16.kicad_sch -> esp-24v-16ch-v6-outputs9-16.kicad_sch
- sheet Output 11: file esp-24v-16ch-v5-outputs9-16.kicad_sch -> esp-24v-16ch-v6-outputs9-16.kicad_sch
- sheet Output 12: file esp-24v-16ch-v5-outputs9-16.kicad_sch -> esp-24v-16ch-v6-outputs9-16.kicad_sch
- sheet Output 13: file esp-24v-16ch-v5-outputs9-16.kicad_sch -> esp-24v-16ch-v6-outputs9-16.kicad_sch
- sheet Output 14: file esp-24v-16ch-v5-outputs9-16.kicad_sch -> esp-24v-16ch-v6-outputs9-16.kicad_sch
- sheet Output 15: file esp-24v-16ch-v5-outputs9-16.kicad_sch -> esp-24v-16ch-v6-outputs9-16.kicad_sch
- sheet Output 16: file esp-24v-16ch-v5-outputs9-16.kicad_sch -> esp-24v-16ch-v6-outputs9-16.kicad_sch
- sheet Output 2: file esp-24v-16ch-v5-outputs1-8.kicad_sch -> esp-24v-16ch-v6-outputs1-8.kicad_sch
- sheet Output 3: file esp-24v-16ch-v5-outputs1-8.kicad_sch -> esp-24v-16ch-v6-outputs1-8.kicad_sch
- sheet Output 4: file esp-24v-16ch-v5-outputs1-8.kicad_sch -> esp-24v-16ch-v6-outputs1-8.kicad_sch
- sheet Output 5: file esp-24v-16ch-v5-outputs1-8.kicad_sch -> esp-24v-16ch-v6-outputs1-8.kicad_sch
- sheet Output 6: file esp-24v-16ch-v5-outputs1-8.kicad_sch -> esp-24v-16ch-v6-outputs1-8.kicad_sch
- sheet Output 7: file esp-24v-16ch-v5-outputs1-8.kicad_sch -> esp-24v-16ch-v6-outputs1-8.kicad_sch
- sheet Output 8: file esp-24v-16ch-v5-outputs1-8.kicad_sch -> esp-24v-16ch-v6-outputs1-8.kicad_sch
- sheet Output 9: file esp-24v-16ch-v5-outputs9-16.kicad_sch -> esp-24v-16ch-v6-outputs9-16.kicad_sch
- sheet Power: file esp-24v-16ch-v5-power.kicad_sch -> esp-24v-16ch-v6-power.kicad_sch
- moved on the sheet: J1, J3, J4, J5

Commit message: Included test points
Parts:
- FID1, FID2, FID3, FID4: JLCPCB BOM (none) -> 0; now in the parts list
- J1: value ENTRADAS 1-8 -> 250-208
- J2: value GNDIO -> 250-202
- J3: value ENTRADAS 9-16 -> 250-208
- J4: value SAÍDAS 1-8 -> 250-208
- J5: value SAÍDAS 9-16 -> 250-208
Other:
- note added: "GNDIO"
- note added: "INPUTS 1-8"
- note added: "INPUTS 9-16"
- note added: "OUTPUTS 1-8"
- note added: "OUTPUTS 9-16"
Changed lines of the file:
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@@
 		(rev "V6.0")
 	)
+	(text "OUTPUTS\n1-8"
+		(exclude_from_sim no)
+		(at 285.75 205.74 0)
+		(effects
+			(font
+				(size 2.5 2.5)
+			)
+			(justify left bottom)
+		)
+	)
+	(text "OUTPUTS\n9-16"
+		(exclude_from_sim no)
+		(at 382.27 205.74 0)
+		(effects
+			(font
+				(size 2.5 2.5)
+			)
+			(justify left bottom)
+		)
+	)
 	(text "RESISTORS: 62,5mW WHERE NOT SPECIFIED"
 		(exclude_from_sim no)
@@
 		)
 	)
+	(text "INPUTS\n1-8"
+		(exclude_from_sim no)
+		(at 24.13 205.74 0)
+		(effects
+			(font
+				(size 2.5 2.5)
+			)
+			(justify left bottom)
+		)
+	)
+	(text "GNDIO"
+		(exclude_from_sim no)
+		(at 26.67 267.97 0)
+		(effects
+			(font
+				(size 2.5 2.5)
+			)
+			(justify left bottom)
+		)
+	)
+	(text "INPUTS\n9-16"
+		(exclude_from_sim no)
+		(at 118.11 205.74 0)
+		(effects
+			(font
+				(size 2.5 2.5)
+			)
+			(justify left bottom)
+		)
+	)
 	(junction
 		(at 45.72 259.08)
@@
 		(body_style 1)
 		(exclude_from_sim no)
-		(in_bom no)
+		(in_bom yes)
 		(on_board yes)
 		(in_pos_files yes)
@@
 			)
 		)
+		(property "JLCPCB BOM" "0"
+			(at 342.9 38.1 0)
+			(hide yes)
+			(show_name no)
+			(do_not_autoplace no)
+			(effects
+				(font
+					(size 1.27 1.27)
+				)
+			)
+		)
 		(instances
 			(project "esp-24v-16ch-v6"
@@
 		(body_style 1)
 		(exclude_from_sim no)
-		(in_bom no)
+		(in_bom yes)
 		(on_board yes)
 		(in_pos_files yes)
@@
 			)
 		)
+		(property "JLCPCB BOM" "0"
+			(at 342.9 44.45 0)
+			(hide yes)
+			(show_name no)
+			(do_not_autoplace no)
+			(effects
+				(font
+					(size 1.27 1.27)
+				)
+			)
+		)
 		(instances
 			(project "esp-24v-16ch-v6"
@@
 			)
 		)
-		(property "Value" "SAÍDAS 9-16"
+		(property "Value" "250-208"
 			(at 386.08 187.9599 0)
 			(show_name no)
@@
 			)
 		)
-		(property "Value" "SAÍDAS 1-8"
+		(property "Value" "250-208"
 			(at 289.56 187.9599 0)
 			(show_name no)
@@
 		(fields_autoplaced yes)
 		(property "Reference" "J3"
-			(at 128.27 185.4199 0)
+			(at 130.81 171.45 0)
 			(show_name no)
 			(do_not_autoplace no)
@@
 					(size 1.27 1.27)
 				)
-				(justify left)
 			)
 		)
-		(property "Value" "ENTRADAS 9-16"
-			(at 128.27 187.9599 0)
+		(property "Value" "250-208"
+			(at 130.81 173.99 0)
 			(show_name no)
 			(do_not_autoplace no)
@@
 					(size 1.27 1.27)
 				)
-				(justify left)
 			)
 		)
@@
 		(body_style 1)
 		(exclude_from_sim no)
-		(in_bom no)
+		(in_bom yes)
 		(on_board yes)
 		(in_pos_files yes)
@@
 			)
 		)
+		(property "JLCPCB BOM" "0"
+			(at 342.9 57.15 0)
+			(hide yes)
+			(show_name no)
+			(do_not_autoplace no)
+			(effects
+				(font
+					(size 1.27 1.27)
+				)
+			)
+		)
 		(instances
 			(project "esp-24v-16ch-v6"
@@
 		(body_style 1)
 		(exclude_from_sim no)
-		(in_bom no)
+		(in_bom yes)
 		(on_board yes)
 		(in_pos_files yes)
@@
 			)
 		)
+		(property "JLCPCB BOM" "0"
+			(at 342.9 50.8 0)
+			(hide yes)
+			(show_name no)
+			(do_not_autoplace no)
+			(effects
+				(font
+					(size 1.27 1.27)
+				)
+			)
+		)
 		(instances
 			(project "esp-24v-16ch-v6"
@@
 		(fields_autoplaced yes)
 		(property "Reference" "J1"
-			(at 34.29 185.4199 0)
+			(at 36.83 171.45 0)
 			(show_name no)
 			(do_not_autoplace no)
@@
 					(size 1.27 1.27)
 				)
-				(justify left)
 			)
 		)
-		(property "Value" "ENTRADAS 1-8"
-			(at 34.29 187.9599 0)
+		(property "Value" "250-208"
+			(at 36.83 173.99 0)
 			(show_name no)
 			(do_not_autoplace no)
@@
 					(size 1.27 1.27)
 				)
-				(justify left)
 			)
 		)
@@
 			)
 		)
-		(property "Value" "GNDIO"
+		(property "Value" "250-202"
 			(at 36.83 255.27 0)
 			(show_name no)

Commit message: Added voltage monitors for both ESP32 and LAN8710A
Parts:
- renumbered J3 to J2, J4 to J3, J5 to J4, J2 to J5
Changed lines of the file:
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@@
 	(title_block
 		(title "ESP 24V 16xIn/16xOut/1-Wire Module")
-		(date "2026-06-01")
-		(rev "V6.0")
+		(date "2026-06-09")
+		(rev "V6.0.3")
 	)
 	(text "OUTPUTS\n1-8"
@@
 		(dnp no)
 		(fields_autoplaced yes)
-		(property "Reference" "J5"
+		(property "Reference" "J4"
 			(at 386.08 185.4199 0)
 			(show_name no)
@@
 			(project "esp-24v-16ch-v6"
 				(path "/2bc5a21a-1d79-419d-a592-6852cc07b00a"
-					(reference "J5")
+					(reference "J4")
 					(unit 1)
 				)
@@
 		(dnp no)
 		(fields_autoplaced yes)
-		(property "Reference" "J4"
+		(property "Reference" "J3"
 			(at 289.56 185.4199 0)
 			(show_name no)
@@
 			(project "esp-24v-16ch-v6"
 				(path "/2bc5a21a-1d79-419d-a592-6852cc07b00a"
-					(reference "J4")
+					(reference "J3")
 					(unit 1)
 				)
@@
 		(dnp no)
 		(fields_autoplaced yes)
-		(property "Reference" "J3"
+		(property "Reference" "J2"
 			(at 130.81 171.45 0)
 			(show_name no)
@@
 			(project "esp-24v-16ch-v6"
 				(path "/2bc5a21a-1d79-419d-a592-6852cc07b00a"
-					(reference "J3")
+					(reference "J2")
 					(unit 1)
 				)
@@
 		(dnp no)
 		(fields_autoplaced yes)
-		(property "Reference" "J2"
+		(property "Reference" "J5"
 			(at 36.83 252.73 0)
 			(show_name no)
@@
 			(project "esp-24v-16ch-v6"
 				(path "/2bc5a21a-1d79-419d-a592-6852cc07b00a"
-					(reference "J2")
+					(reference "J5")
 					(unit 1)
 				)
