File: V6/eumesmo-io-24v16ch-v6-lan.kicad_sch (KiCad schematic)
At the start: 29 parts, among them J8 ETHERNET, U6 LAN8710A, U7 TPS3823-33

Commit message: Renamed all files to eumesmo branding
Other:
- title: ESP 24V 16xIn/16xOut/1-Wire Module -> eumesmo 24V 16xIn/16xOut/1-Wire Module

Commit message: Added CPU health LED
Parts:
- renumbered C25 to C19, C24 to C20, C19 to C21, C20 to C22, C21 to C23, C22 to C24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
