File: V6/eumesmo-io-24v16ch-v6-lan.kicad_sch (KiCad schematic)
At the start: 29 parts, among them J8 ETHERNET, U6 LAN8710A, U7 TPS3820-33

Commit message: Remove jumpers from BOM.
Parts:
- D8: FT Rotation Offset 0 -> 90
- J8, U6: FT Rotation Offset 0 -> 180
Changed lines of the file:
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@@
 			)
 		)
-		(property "FT Rotation Offset" "0"
+		(property "FT Rotation Offset" "180"
 			(at 48.26 154.94 0)
 			(hide yes)
@@
 			)
 		)
-		(property "FT Rotation Offset" "0"
+		(property "FT Rotation Offset" "90"
 			(at 252.73 93.98 0)
 			(hide yes)
@@
 			)
 		)
-		(property "FT Rotation Offset" "0"
+		(property "FT Rotation Offset" "180"
 			(at 176.53 88.9 0)
 			(hide yes)
