File: V6/eumesmo-io-24v16ch-v6.kicad_pcb (KiCad board)
At the start: 4 copper layers, 128 x 67.8 mm, 335 parts, among them J1 250-208, J2 250-208, J3 250-208, J4 250-208, J5 250-202, J6 250-202, J7 USB_C_Receptacle_USB2.0, J8 ETHERNET, J9 250-203, Q1 WPM2015-3/TR, Q10 MMBT2222A, Q11 MMBT2222A, Q12 MMBT2222A, Q13 MMBT2222A, Q14 MMBT2222A, Q15 MMBT2222A, Q16 MMBT2222A, Q17 MMBT2222A, Q18 MMBT2222A, Q19 MMBT2222A, Q2 MMUN2211LT3G, Q3 UMH3N, Q4 MMBT2222A, Q5 MMBT2222A, Q6 MMBT2222A, Q7 MMBT2222A, Q8 MMBT2222A, Q9 MMBT2222A, SW1 RESET, SW2 1WIRE_SEL, U1 TX4138, U10 MCP23017, U11 DS2482S-100, U12 OR-3H7-4, U13 OR-3H7-4, U14 OR-3H7-4, U15 OR-3H7-4, U2 SY8089A1AAC, U3 TPS3820-33, U4 CH340K, U5 ESP32-WROOM-32UE-N16, U6 LAN8710A, U7 TPS3820-33, U8 MCP23008, U9 MCP23008

Commit message: LEDs changed to orange
Parts:
- D13, D16, D19, D22, D25, D28, D31, D34, D37, D40, D43, D46, D49, D52, D55, D58, D59, D6, D60, D61, D62, D63, D64, D65, D66, D67, D68, D69, D7, D70, D71, D72, D73, D74: value EMERALD/0603 -> ORANGE/0603
- R102, R105, R108, R111, R114, R117, R120, R123, R126, R129, R132, R135, R44, R47, R50, R53, R56, R59, R62, R65, R68, R71, R74, R77, R80, R83, R86, R89, R90, R93, R96, R99: value 10k/125mW -> 9.1k/125mW
- R11, R13: value 330R -> 680R

Commit message: LEDs replaced for orange
Parts:
- R102, R105, R108, R111, R114, R117, R120, R123, R126, R129, R132, R135, R44, R47, R50, R53, R56, R59, R62, R65, R68, R71, R74, R77, R80, R83, R86, R89, R90, R93, R96, R99: value 9.1k/125mW -> 10k/125mW
