File: V6/eumesmo-io-24v16ch-v6-i2c.kicad_sch (KiCad schematic)
At the start: 25 parts, among them J9 250-203, SW2 1WIRE_SEL, U10 MCP23017, U11 DS2482S-100, U8 MCP23008, U9 MCP23008

Commit message: Further improvements to routing between ETH jack and LAN IC.
Parts:
- JP1: now not fitted
Changed lines of the file:
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@@
 		(exclude_from_sim no)
 		(in_bom no)
-		(on_board yes)
+		(on_board no)
 		(in_pos_files yes)
-		(dnp no)
+		(dnp yes)
 		(fields_autoplaced yes)
 		(property "Reference" "JP1"

Commit message: Remove jumpers from BOM.
Parts:
- SW2, U11: FT Rotation Offset 0 -> 270
Changed lines of the file:
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@@
 			)
 		)
-		(property "FT Rotation Offset" "0"
+		(property "FT Rotation Offset" "270"
 			(at 245.11 186.69 0)
 			(hide yes)
@@
 			)
 		)
-		(property "FT Rotation Offset" "0"
-			(at 285.75 166.37 0)
-			(hide yes)
+		(property "FT Rotation Offset" "270"
+			(at 285.75 166.37 0)
+			(hide yes)

Commit message: Adjusted component rotation and offset information for JLCPCB.
Parts:
- SW2, U11: FT Rotation Offset 270 -> -90
Changed lines of the file:
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@@
 			)
 		)
+		(property "FT Position Offset" ""
+			(at 83.82 73.66 0)
+			(hide yes)
+			(show_name no)
+			(do_not_autoplace no)
+			(effects
+				(font
+					(size 1.27 1.27)
+				)
+			)
+		)
 		(pin "3"
 		)
@@
 			)
 		)
-		(property "Package" ""
+		(property "Case" "0402/1005"
 			(at 162.56 191.77 0)
 			(hide yes)
@@
 			)
 		)
-		(property "Case" "0402/1005"
+		(property "FT Rotation Offset" "0"
 			(at 162.56 191.77 0)
 			(hide yes)
@@
 			)
 		)
-		(property "FT Rotation Offset" "0"
+		(property "FT Position Offset" ""
 			(at 162.56 191.77 0)
 			(hide yes)
@@
 			)
 		)
+		(property "FT Position Offset" ""
+			(at 135.89 185.42 0)
+			(hide yes)
+			(show_name no)
+			(do_not_autoplace no)
+			(effects
+				(font
+					(size 1.27 1.27)
+				)
+			)
+		)
 		(pin "3"
 		)
@@
 			)
 		)
+		(property "FT Position Offset" ""
+			(at 195.58 185.42 90)
+			(hide yes)
+			(show_name no)
+			(do_not_autoplace no)
+			(effects
+				(font
+					(size 1.27 1.27)
+				)
+			)
+		)
 		(pin "2"
 		)
@@
 			)
 		)
-		(property "Package" ""
+		(property "Case" "0805/2012"
 			(at 246.38 148.59 0)
 			(hide yes)
@@
 			)
 		)
-		(property "Case" "0805/2012"
+		(property "FT Rotation Offset" "0"
 			(at 246.38 148.59 0)
 			(hide yes)
@@
 			)
 		)
-		(property "FT Rotation Offset" "0"
+		(property "FT Position Offset" ""
 			(at 246.38 148.59 0)
 			(hide yes)
@@
 			)
 		)
-		(property "Package" ""
+		(property "Case" "0805/2012"
 			(at 148.59 191.77 0)
 			(hide yes)
@@
 			)
 		)
-		(property "Case" "0805/2012"
+		(property "FT Rotation Offset" "0"
 			(at 148.59 191.77 0)
 			(hide yes)
@@
 			)
 		)
-		(property "FT Rotation Offset" "0"
+		(property "FT Position Offset" ""
 			(at 148.59 191.77 0)
 			(hide yes)
@@
 			)
 		)
+		(property "FT Position Offset" ""
+			(at 245.11 199.39 0)
+			(hide yes)
+			(show_name no)
+			(do_not_autoplace no)
+			(effects
+				(font
+					(size 1.27 1.27)
+				)
+			)
+		)
 		(pin "2"
 		)
@@
 			)
 		)
+		(property "FT Position Offset" ""
+			(at 163.83 57.15 0)
+			(hide yes)
+			(show_name no)
+			(do_not_autoplace no)
+			(effects
+				(font
+					(size 1.27 1.27)
+				)
+			)
+		)
 		(pin "1"
 		)
@@
 			)
 		)
+		(property "FT Position Offset" ""
+			(at 345.44 85.09 0)
+			(hide yes)
+			(show_name no)
+			(do_not_autoplace no)
+			(effects
+				(font
+					(size 1.27 1.27)
+				)
+			)
+		)
 		(pin "1"
 		)
@@
 			)
 		)
+		(property "FT Position Offset" ""
+			(at 57.15 57.15 0)
+			(hide yes)
+			(show_name no)
+			(do_not_autoplace no)
+			(effects
+				(font
+					(size 1.27 1.27)
+				)
+			)
+		)
 		(pin "1"
 		)
@@
 			)
 		)
+		(property "FT Position Offset" ""
+			(at 91.44 45.72 0)
+			(hide yes)
+			(show_name no)
+			(do_not_autoplace no)
+			(effects
+				(font
+					(size 1.27 1.27)
+				)
+			)
+		)
 		(pin "1"
 		)
@@
 			)
 		)
+		(property "FT Position Offset" ""
+			(at 203.2 176.53 0)
+			(hide yes)
+			(show_name no)
+			(do_not_autoplace no)
+			(effects
+				(font
+					(size 1.27 1.27)
+				)
+			)
+		)
 		(pin "1"
 		)
@@
 			)
 		)
+		(property "FT Position Offset" ""
+			(at 198.12 45.72 0)
+			(hide yes)
+			(show_name no)
+			(do_not_autoplace no)
+			(effects
+				(font
+					(size 1.27 1.27)
+				)
+			)
+		)
 		(pin "1"
 		)
@@
 			)
 		)
+		(property "FT Position Offset" ""
+			(at 175.26 191.77 90)
+			(hide yes)
+			(show_name no)
+			(do_not_autoplace no)
+			(effects
+				(font
+					(size 1.27 1.27)
+				)
+			)
+		)
 		(pin "1"
 		)
@@
 			)
 		)
-		(property "Package" ""
+		(property "Case" "0402/1005"
 			(at 278.13 148.59 0)
 			(hide yes)
@@
 			)
 		)
-		(property "Case" "0402/1005"
+		(property "FT Rotation Offset" "0"
 			(at 278.13 148.59 0)
 			(hide yes)
@@
 			)
 		)
-		(property "FT Rotation Offset" "0"
+		(property "FT Position Offset" ""
 			(at 278.13 148.59 0)
 			(hide yes)
@@
 			)
 		)
+		(property "FT Position Offset" ""
+			(at 203.2 191.77 0)
+			(hide yes)
+			(show_name no)
+			(do_not_autoplace no)
+			(effects
+				(font
+					(size 1.27 1.27)
+				)
+			)
+		)
 		(pin "1"
 		)
@@
 			)
 		)
+		(property "FT Position Offset" ""
+			(at 345.44 67.31 0)
+			(hide yes)
+			(show_name no)
+			(do_not_autoplace no)
+			(effects
+				(font
+					(size 1.27 1.27)
+				)
+			)
+		)
 		(pin "1"
 		)
@@
 			)
 		)
+		(property "FT Position Offset" ""
+			(at 190.5 73.66 0)
+			(hide yes)
+			(show_name no)
+			(do_not_autoplace no)
+			(effects
+				(font
+					(size 1.27 1.27)
+				)
+			)
+		)
 		(pin "3"
 		)
@@
 			)
 		)
+		(property "FT Position Offset" ""
+			(at 187.96 191.77 90)
+			(hide yes)
+			(show_name no)
+			(do_not_autoplace no)
+			(effects
+				(font
+					(size 1.27 1.27)
+				)
+			)
+		)
 		(pin "1"
 		)
@@
 			)
 		)
+		(property "FT Position Offset" ""
+			(at 278.13 83.82 0)
+			(hide yes)
+			(show_name no)
+			(do_not_autoplace no)
+			(effects
+				(font
+					(size 1.27 1.27)
+				)
+			)
+		)
 		(pin "4"
 		)
@@
 			)
 		)
+		(property "FT Position Offset" ""
+			(at 250.19 80.01 0)
+			(hide yes)
+			(show_name no)
+			(do_not_autoplace no)
+			(effects
+				(font
+					(size 1.27 1.27)
+				)
+			)
+		)
 		(pin "1"
 		)
@@
 			)
 		)
-		(property "FT Rotation Offset" "270"
+		(property "FT Rotation Offset" "-90"
+			(at 245.11 186.69 0)
+			(hide yes)
+			(show_name no)
+			(do_not_autoplace no)
+			(effects
+				(font
+					(size 1.27 1.27)
+				)
+			)
+		)
+		(property "FT Position Offset" ""
 			(at 245.11 186.69 0)
 			(hide yes)
@@
 			)
 		)
+		(property "FT Position Offset" ""
+			(at 285.75 45.72 0)
+			(hide yes)
+			(show_name no)
+			(do_not_autoplace no)
+			(effects
+				(font
+					(size 1.27 1.27)
+				)
+			)
+		)
 		(pin "1"
 		)
@@
 			)
 		)
-		(property "FT Rotation Offset" "270"
+		(property "FT Rotation Offset" "-90"
+			(at 285.75 166.37 0)
+			(hide yes)
+			(show_name no)
+			(do_not_autoplace no)
+			(effects
+				(font
+					(size 1.27 1.27)
+				)
+			)
+		)
+		(property "FT Position Offset" ""
 			(at 285.75 166.37 0)
 			(hide yes)
@@
 			)
 		)
-		(property "Package" ""
+		(property "Case" "0805/2012"
 			(at 304.8 45.72 0)
 			(hide yes)
@@
 			)
 		)
-		(property "Case" "0805/2012"
+		(property "FT Rotation Offset" "0"
 			(at 304.8 45.72 0)
 			(hide yes)
@@
 			)
 		)
-		(property "FT Rotation Offset" "0"
+		(property "FT Position Offset" ""
 			(at 304.8 45.72 0)
 			(hide yes)

Commit message: Connectors moved up into the board.
Parts:
- C30, C31, SW2, U11: now not fitted; now left out of the parts list
- JP1: footprint Jumper:SolderJumper-2_P1.3mm_Open_RoundedPad1.0x1.5mm -> Jumper:SolderJumper-2_P1.3mm_Bridged_RoundedPad1.0x1.5mm
Other:
- note added: "ATTENTION! DIP SWITCH SW2: ONLY ONE SWITCH CAN BE ON AT ANY GIVEN TIME. JUMPER JP1: BRIDGED BY DEFAULT. MUST BE CUT TO USE DS2482 WHEN POPULATED."
- note removed: "ATTENTION! DIP SWITCH SW2: ONLY ONE SWITCH CAN BE ON AT ANY GIVEN TIME. JUMPER JP1: MUST BE CLOSED TO CONNECT 1-WIRE INPUT TO GPIO16 WHEN THE SWITCH AND DS2482 ARE NOT POPULATED."
