File: V6/eumesmo-io-24v16ch-v6.kicad_sch (KiCad schematic)
At the start: 9 parts, among them J1 250-208, J2 250-208, J3 250-208, J4 250-208, J5 250-202

Commit message: Replaced Wago connectors for other brand, no stock.
Parts:
- J1, J2, J3, J4: LCSC Part # C2833587 -> C475160; Mfr Wago -> Cixi Kefa Elec; Mfr PN 250-208 -> KF250-3.5-8P-1; Vendor PN C2833587 -> C475160
- J5: LCSC Part # C2765061 -> C475154; Mfr Wago -> Cixi Kefa Elec; Mfr PN 250-202 -> KF250-3.5-2P-1; Vendor PN C2765061 -> C475154
Changed lines of the file:
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@@
 			)
 		)
-		(property "LCSC Part #" "C2833587"
+		(property "LCSC Part #" "C475160"
 			(at 383.54 185.42 0)
 			(hide yes)
@@
 			)
 		)
-		(property "Mfr" "Wago"
+		(property "Mfr" "Cixi Kefa Elec"
 			(at 383.54 185.42 0)
 			(hide yes)
@@
 			)
 		)
-		(property "Mfr PN" "250-208"
+		(property "Mfr PN" "KF250-3.5-8P-1"
 			(at 383.54 185.42 0)
 			(hide yes)
@@
 			)
 		)
-		(property "Vendor PN" "C2833587"
+		(property "Vendor PN" "C475160"
 			(at 383.54 185.42 0)
 			(hide yes)
@@
 			)
 		)
-		(property "LCSC Part #" "C2833587"
+		(property "LCSC Part #" "C475160"
 			(at 287.02 185.42 0)
 			(hide yes)
@@
 			)
 		)
-		(property "Mfr" "Wago"
+		(property "Mfr" "Cixi Kefa Elec"
 			(at 287.02 185.42 0)
 			(hide yes)
@@
 			)
 		)
-		(property "Mfr PN" "250-208"
+		(property "Mfr PN" "KF250-3.5-8P-1"
 			(at 287.02 185.42 0)
 			(hide yes)
@@
 			)
 		)
-		(property "Vendor PN" "C2833587"
+		(property "Vendor PN" "C475160"
 			(at 287.02 185.42 0)
 			(hide yes)
@@
 			)
 		)
-		(property "LCSC Part #" "C2833587"
+		(property "LCSC Part #" "C475160"
 			(at 130.81 185.42 0)
 			(hide yes)
@@
 			)
 		)
-		(property "Mfr" "Wago"
+		(property "Mfr" "Cixi Kefa Elec"
 			(at 130.81 185.42 0)
 			(hide yes)
@@
 			)
 		)
-		(property "Mfr PN" "250-208"
+		(property "Mfr PN" "KF250-3.5-8P-1"
 			(at 130.81 185.42 0)
 			(hide yes)
@@
 			)
 		)
-		(property "Vendor PN" "C2833587"
+		(property "Vendor PN" "C475160"
 			(at 130.81 185.42 0)
 			(hide yes)
@@
 			)
 		)
-		(property "LCSC Part #" "C2833587"
+		(property "LCSC Part #" "C475160"
 			(at 36.83 185.42 0)
 			(hide yes)
@@
 			)
 		)
-		(property "Mfr" "Wago"
+		(property "Mfr" "Cixi Kefa Elec"
 			(at 36.83 185.42 0)
 			(hide yes)
@@
 			)
 		)
-		(property "Mfr PN" "250-208"
+		(property "Mfr PN" "KF250-3.5-8P-1"
 			(at 36.83 185.42 0)
 			(hide yes)
@@
 			)
 		)
-		(property "Vendor PN" "C2833587"
+		(property "Vendor PN" "C475160"
 			(at 36.83 185.42 0)
 			(hide yes)
@@
 			)
 		)
-		(property "LCSC Part #" "C2765061"
+		(property "LCSC Part #" "C475154"
 			(at 36.83 259.08 0)
 			(hide yes)
@@
 			)
 		)
-		(property "Mfr" "Wago"
+		(property "Mfr" "Cixi Kefa Elec"
 			(at 36.83 259.08 0)
 			(hide yes)
@@
 			)
 		)
-		(property "Mfr PN" "250-202"
+		(property "Mfr PN" "KF250-3.5-2P-1"
 			(at 36.83 259.08 0)
 			(hide yes)
@@
 			)
 		)
-		(property "Vendor PN" "C2765061"
+		(property "Vendor PN" "C475154"
 			(at 36.83 259.08 0)
 			(hide yes)
